File: hw-design/receiver/bluetooth.sch (KiCad schematic (older format))
At the start: 20 parts, among them U7 nRF8001, Y2 32kHz, Y3 16MHz

Commit message: Revision 2
Parts:
- Y3: footprint w_crystal:hc-49_smd -> w_crystal:crystal_hc-49s
Other:
- note removed: "Ten sam co do µC"
Changed lines of the file:
@@
 $EndComp
 $Comp
-L GND #PWR028
+L GND #PWR036
 U 1 1 56376523
 P 4900 4000
-F 0 "#PWR028" H 4900 3750 50  0001 C CNN
+F 0 "#PWR036" H 4900 3750 50  0001 C CNN
 F 1 "GND" H 4900 3850 50  0000 C CNN
 F 2 "" H 4900 4000 60  0000 C CNN
@@
 $EndComp
 $Comp
-L GND #PWR029
+L GND #PWR037
 U 1 1 56376527
 P 3750 3925
-F 0 "#PWR029" H 3750 3675 50  0001 C CNN
+F 0 "#PWR037" H 3750 3675 50  0001 C CNN
 F 1 "GND" H 3750 3775 50  0000 C CNN
 F 2 "" H 3750 3925 60  0000 C CNN
@@
 Connection ~ 4400 3800
 $Comp
-L +3.3V #PWR030
+L +3.3V #PWR038
 U 1 1 56376528
 P 4975 2650
-F 0 "#PWR030" H 4975 2500 50  0001 C CNN
+F 0 "#PWR038" H 4975 2500 50  0001 C CNN
 F 1 "+3.3V" H 4975 2790 50  0000 C CNN
 F 2 "" H 4975 2650 60  0000 C CNN
@@
 Connection ~ 4975 2725
 $Comp
-L GND #PWR031
+L GND #PWR039
 U 1 1 5637652C
 P 4050 2725
-F 0 "#PWR031" H 4050 2475 50  0001 C CNN
+F 0 "#PWR039" H 4050 2475 50  0001 C CNN
 F 1 "GND" H 4050 2575 50  0000 C CNN
 F 2 "" H 4050 2725 60  0000 C CNN
@@
 $EndComp
 $Comp
-L GND #PWR032
+L GND #PWR040
 U 1 1 5637652D
 P 4050 3000
-F 0 "#PWR032" H 4050 2750 50  0001 C CNN
+F 0 "#PWR040" H 4050 2750 50  0001 C CNN
 F 1 "GND" H 4050 2850 50  0000 C CNN
 F 2 "" H 4050 3000 60  0000 C CNN
@@
 $EndComp
 $Comp
-L GND #PWR033
+L GND #PWR041
 U 1 1 5637652E
 P 4600 2725
-F 0 "#PWR033" H 4600 2475 50  0001 C CNN
+F 0 "#PWR041" H 4600 2475 50  0001 C CNN
 F 1 "GND" H 4600 2575 50  0000 C CNN
 F 2 "" H 4600 2725 60  0000 C CNN
@@
 $EndComp
 $Comp
-L +3.3V #PWR034
+L +3.3V #PWR042
 U 1 1 5637652F
 P 5450 4625
-F 0 "#PWR034" H 5450 4475 50  0001 C CNN
+F 0 "#PWR042" H 5450 4475 50  0001 C CNN
 F 1 "+3.3V" H 5450 4765 50  0000 C CNN
 F 2 "" H 5450 4625 60  0000 C CNN
@@
 	5000 4450 5000 3900
 $Comp
-L GND #PWR035
+L GND #PWR043
 U 1 1 56376531
 P 6725 4275
-F 0 "#PWR035" H 6725 4025 50  0001 C CNN
+F 0 "#PWR043" H 6725 4025 50  0001 C CNN
 F 1 "GND" H 6725 4125 50  0000 C CNN
 F 2 "" H 6725 4275 60  0000 C CNN
@@
 Connection ~ 6725 3900
 $Comp
-L GND #PWR036
+L GND #PWR044
 U 1 1 56376532
 P 5550 2575
-F 0 "#PWR036" H 5550 2325 50  0001 C CNN
+F 0 "#PWR044" H 5550 2325 50  0001 C CNN
 F 1 "GND" H 5550 2425 50  0000 C CNN
 F 2 "" H 5550 2575 60  0000 C CNN
@@
 Connection ~ 5550 2675
 $Comp
-L +3.3V #PWR037
+L +3.3V #PWR045
 U 1 1 56376533
 P 5750 2600
-F 0 "#PWR037" H 5750 2450 50  0001 C CNN
+F 0 "#PWR045" H 5750 2450 50  0001 C CNN
 F 1 "+3.3V" H 5750 2740 50  0000 C CNN
 F 2 "" H 5750 2600 60  0000 C CNN
@@
 F 0 "Y3" H 5925 2275 50  0000 C CNN
 F 1 "16MHz" H 5925 1975 50  0000 C CNN
-F 2 "w_crystal:hc-49_smd" H 5925 2125 60  0001 C CNN
+F 2 "w_crystal:crystal_hc-49s" H 5925 2125 60  0001 C CNN
 F 3 "http://pl.farnell.com/abracon/abm8-16-000mhz-10-1-u-t/crystal-16mhz-10pf-3-2-x-2-5mm/dp/2467830" H 5925 2125 60  0001 C CNN
 F 4 "Kryształ 16MHz do radia do nRF8001" H 5925 2125 60  0001 C CNN "Opis"
@@
 Connection ~ 6200 1500
 $Comp
-L GND #PWR038
+L GND #PWR046
 U 1 1 56376537
 P 6325 1500
-F 0 "#PWR038" H 6325 1250 50  0001 C CNN
+F 0 "#PWR046" H 6325 1250 50  0001 C CNN
 F 1 "GND" H 6325 1350 50  0000 C CNN
 F 2 "" H 6325 1500 60  0000 C CNN
@@
 	0    -1   -1   0
 $EndComp
-Text Notes 4750 2150 0    60   ~ 0
-Ten sam co do µC
-$Comp
-L +3.3V #PWR039
+$Comp
+L +3.3V #PWR047
 U 1 1 56376538
 P 6975 2150
-F 0 "#PWR039" H 6975 2000 50  0001 C CNN
+F 0 "#PWR047" H 6975 2000 50  0001 C CNN
 F 1 "+3.3V" H 6975 2290 50  0000 C CNN
 F 2 "" H 6975 2150 60  0000 C CNN
@@
 $EndComp
 $Comp
-L GND #PWR040
+L GND #PWR048
 U 1 1 5637653B
 P 6975 2775
-F 0 "#PWR040" H 6975 2525 50  0001 C CNN
+F 0 "#PWR048" H 6975 2525 50  0001 C CNN
 F 1 "GND" H 6975 2625 50  0000 C CNN
 F 2 "" H 6975 2775 60  0000 C CNN
@@
 	6600 3200 6725 3200
 $Comp
-L +3.3V #PWR041
+L +3.3V #PWR049
 U 1 1 5637653C
 P 6725 3200
-F 0 "#PWR041" H 6725 3050 50  0001 C CNN
+F 0 "#PWR049" H 6725 3050 50  0001 C CNN
 F 1 "+3.3V" H 6725 3340 50  0000 C CNN
 F 2 "" H 6725 3200 60  0000 C CNN
@@
 $EndComp
 $Comp
-L GND #PWR042
+L GND #PWR050
 U 1 1 5637653D
 P 6900 3300
-F 0 "#PWR042" H 6900 3050 50  0001 C CNN
+F 0 "#PWR050" H 6900 3050 50  0001 C CNN
 F 1 "GND" H 6900 3150 50  0000 C CNN
 F 2 "" H 6900 3300 60  0000 C CNN
@@
 Connection ~ 8700 3050
 $Comp
-L GND #PWR043
+L GND #PWR051
 U 1 1 56376543
 P 8700 3600
-F 0 "#PWR043" H 8700 3350 50  0001 C CNN
+F 0 "#PWR051" H 8700 3350 50  0001 C CNN
 F 1 "GND" H 8700 3450 50  0000 C CNN
 F 2 "" H 8700 3600 60  0000 C CNN
@@
 	8350 3800 8350 3975
 $Comp
-L GND #PWR044
+L GND #PWR052
 U 1 1 56376545
 P 8350 4375
-F 0 "#PWR044" H 8350 4125 50  0001 C CNN
+F 0 "#PWR052" H 8350 4125 50  0001 C CNN
 F 1 "GND" H 8350 4225 50  0000 C CNN
 F 2 "" H 8350 4375 60  0000 C CNN
