File: hw-design/receiver/gp8-clock.kicad_pcb (KiCad board)
At the start: 2 copper layers, 103.8 x 50.9 mm, 82 parts, among them P1 CONN_01X03, Q1 Q_NPN_BCE, Q2 Q_NPN_BCE, SW1 SW_PUSH, SW2 power, U1 TSOP39538, U2 weight-scale-lcd, U3 STM32F0-LQFP48, U4 usb-micro, U5 MCP73833, U6 AP1117D33, U7 nRF8001, Y1 Crystal, Y2 32kHz, Y3 16MHz

Commit message: Skończona rewizja r1, wysłane do satlanfd
Parts:
- R25, R26, R27: value 560R -> 730R
- SW2: footprint w_switch:PCB_PUSH -> w_pin_strip:pin_socket_2
Routing:
- net Net-(P1-Pad1): track 24.1 -> 19.9 mm
- net GND: track 811.8 -> 809.8 mm
- net /seg2: track 11.7 -> 12.8 mm
- net /com1: track 28.3 -> 29.2 mm
- net /com3: track 22.3 -> 23.1 mm
- net Net-(C16-Pad1): track 41.0 -> 40.3 mm
- net /seg4: track 10.2 -> 10.8 mm
- net /com4: track 19.1 -> 19.7 mm
- net +5V: track 39.2 -> 39.8 mm

Commit message: Revision 2
Parts:
- removed D3: LED, w_indicators:led_3mm_yellow
- removed D4: LED, w_indicators:led_3mm_green
- removed D5: LED, w_indicators:led_3mm_red
- added P2: test-double, iwasz:testpad-2p, B.Cu at (131.8, 96.5)
- added P3: CONN_01X04, w_pin_strip:pin_strip_4, B.Cu at (147.3, 125.7)
- added P4: test-double, iwasz:testpad-2p, B.Cu at (194.1, 105.2)
- added P5: test-double, iwasz:testpad-2p, B.Cu at (194.6, 110.7)
- added P6: test-double, iwasz:testpad-2p, B.Cu at (183.4, 107.7)
- added Q3: BC847, w_smd_trans:sot23, B.Cu at (178.3, 123.4)
- added Q4: BC847, w_smd_trans:sot23, B.Cu at (165.6, 119.4)
- added Q5: NX7002AK, iwasz:sot23-pins123-ccw, B.Cu at (157.0, 121.9)
- added R31: 22R, w_smd_resistors:r_0603, B.Cu at (146.3, 122.4)
- added R32: 22R, w_smd_resistors:r_0603, B.Cu at (151.4, 122.4)
- added R33: 1k, w_smd_resistors:r_0603, B.Cu at (169.7, 118.4)
- added R34: 10k, w_smd_resistors:r_0603, B.Cu at (161.0, 120.4)
- added SP1: BUZZER, Buzzers_Beepers:Buzzer_12x9.5RM7.6, B.Cu at (186.1, 119.4)
- C15, C16, C17: footprint w_smd_cap:c_tant_A -> w_smd_cap:c_tant_B
- D2: footprint w_indicators:led_3mm_red -> w_indicators:led_5mm_red
- P1: footprint w_conn_df13:df13-3p-125dsa -> w_pin_strip:pin_strip_3
- Q1, Q2: value Q_NPN_BCE -> BC847
- R25: value 730R -> Photores; footprint w_smd_resistors:r_0603 -> photo-elements:T0-46-A10XX; moved to F.Cu
- R26: value 730R -> 10k
- R27: value 730R -> 1k
- SW1: footprint w_switch:PCB_PUSH -> iwasz:tact-switch-smd
- SW2: footprint w_pin_strip:pin_socket_2 -> w_pin_strip:pin_strip_2; moved to B.Cu
- Y1, Y3: footprint w_crystal:hc-49_smd -> w_crystal:crystal_hc-49s
- moved R27 35.0 mm to (175.3, 123.4)
- moved R26 27.2 mm to (174.8, 115.8), turned to 0 degrees
- moved SW2 26.6 mm to (156.2, 118.1)
- moved SW1 21.5 mm to (185.4, 94.5), turned to 180 degrees
- moved C12 20.4 mm to (178.8, 94.5), turned to 270 degrees
- moved R25 16.8 mm to (174.6, 111.1), turned to 270 degrees
- moved C22 15.6 mm to (128.3, 113.0), turned to 180 degrees
- moved C4 6.35 mm to (144.8, 109.9)
- moved R22 6.23 mm to (141.6, 109.9)
- moved R29 4.89 mm to (120.9, 109.2), turned to 180 degrees
- moved Y1 3.91 mm to (141.6, 114.3)
- moved C26 3.70 mm to (127.5, 100.6)
- moved C14 2.96 mm to (146.8, 96.5)
- moved U6 2.87 mm to (155.6, 104.8)
- moved C6 2.54 mm to (126.0, 97.0)
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Connections:
- C16 pad 1: Net-(C16-Pad1) -> +BATT
- P1 pad 2: GND -> Net-(P1-Pad2)
- P1 pad 3: Net-(P1-Pad3) -> GND
- R25 pad 1: Net-(D3-Pad1) -> +3V3
- R26 pad 1: Net-(D4-Pad1) -> Net-(R25-Pad2)
- R26 pad 2: Net-(R26-Pad2) -> GND
- R27 pad 1: Net-(D5-Pad1) -> /sound
- R27 pad 2: Net-(R27-Pad2) -> Net-(Q3-Pad1)
- R30 pad 1: Net-(R30-Pad1) -> (no net)
- SW2 pad 2: Net-(C16-Pad1) -> +BATT
- U3 pad 1: Net-(U3-Pad1) -> (no net)
- U3 pad 2: Net-(U3-Pad2) -> complete
- U3 pad 3: Net-(U3-Pad3) -> Net-(R25-Pad2)
- U3 pad 34: /seg7 -> /swdio
- U3 pad 35: Net-(U3-Pad35) -> GND
- U3 pad 37: /seg8 -> /swdclk
- U3 pad 38: /seg9 -> /seg7
- U3 pad 39: /seg10 -> /seg8
- U3 pad 4: Net-(U3-Pad4) -> /sound
- U3 pad 40: /seg11 -> /seg9
- U3 pad 41: /seg12 -> /seg10
- U3 pad 42: Net-(C12-Pad1) -> /seg11
- U3 pad 43: Net-(U3-Pad43) -> /seg12
- U3 pad 44: Net-(U3-Pad44) -> (no net)
- U3 pad 45: Net-(U3-Pad45) -> Net-(C12-Pad1)
- U3 pad 46: Net-(U3-Pad46) -> progress
- U4 pad 4: Net-(U4-Pad4) -> (no net)
- U5 pad 3: Net-(R27-Pad2) -> progress
- U5 pad 4: Net-(R26-Pad2) -> complete
- U5 pad 7: Net-(R25-Pad2) -> Net-(P6-Pad1)
- U5 pad 8: Net-(P1-Pad3) -> Net-(P1-Pad2)
- U6 pad 3: Net-(C16-Pad1) -> +BATT
- U7 pad 10: Net-(U7-Pad10) -> (no net)
- U7 pad 15: Net-(U7-Pad15) -> (no net)
- U7 pad 32: Net-(U7-Pad32) -> (no net)
- U7 pad 7: Net-(U7-Pad7) -> (no net)
Routing:
- net GND: track 809.8 -> 1143.3 mm, vias 196 -> 233
- net complete: track 0.00 -> 66.1 mm, vias 0 -> 2
- net progress: track 0.00 -> 61.7 mm, vias 0 -> 2
- net /sound: track 0.00 -> 43.8 mm, vias 0 -> 2
- net Net-(C16-Pad1): track 40.3 -> 0.00 mm
- net /swdio: track 0.00 -> 37.6 mm, vias 0 -> 2
- net /swdclk: track 0.00 -> 34.8 mm, vias 0 -> 2
- net Net-(R25-Pad2): track 8.41 -> 41.7 mm
- net +BATT: track 38.0 -> 69.8 mm
- net Net-(P6-Pad1): track 0.00 -> 29.5 mm
- net +5V: track 39.8 -> 17.0 mm
- net Net-(R26-Pad2): track 20.5 -> 0.00 mm
- net Net-(P1-Pad1): track 19.9 -> 40.1 mm
- net +3V3: track 165.3 -> 183.7 mm, vias 16 -> 14
- net Net-(R27-Pad2): track 17.8 -> 0.00 mm
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Other:
- board size 103.8 x 50.9 mm -> 102.3 x 50.9 mm
- net class Default: trace_width 0.1524 -> 0.2032
- board text added: "Iwasz 2016"
- board text added: "facing ground"
- board text added: "facing sky"
- board text added: "moto-gymkhana stopwatch by iwasz. rev2. 2016"
- board text removed: "current 300mA"
- board text removed: "moto-gymkhana stopwatch by iwasz. rev1. 2015"

Commit message: Funkcjonaloność tego zegara na LEDac jest w tym momencie powtórzona na LCDku
Other:
- board text added: "+"
- board text added: "-"
- board text added: "3v3"
- board text added: "clk"
- board text added: "gnd"
- board text added: "io"
Changed lines of the file:
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@@
     (area 87.000001 76.946 205.400001 137.300001)
     (thickness 1.6)
-    (drawings 220)
+    (drawings 226)
     (tracks 1564)
     (zones 0)
@@
     )
   )
+  (gr_text clk (at 152.908 122.428 90) (layer B.SilkS)
+    (effects (font (size 1.016 1.016) (thickness 0.127)))
+  )
+  (gr_text gnd (at 147.828 122.936 90) (layer B.SilkS)
+    (effects (font (size 1.016 1.016) (thickness 0.127)))
+  )
+  (gr_text io (at 145.796 119.38 90) (layer B.SilkS)
+    (effects (font (size 1.016 1.016) (thickness 0.127)))
+  )
+  (gr_text 3v3 (at 142.748 122.936 90) (layer B.SilkS)
+    (effects (font (size 1.016 1.016) (thickness 0.127)))
+  )
+  (gr_text + (at 180.848 98.552) (layer B.SilkS)
+    (effects (font (size 1.5 1.5) (thickness 0.3)))
+  )
+  (gr_text - (at 180.848 106.172) (layer B.SilkS)
+    (effects (font (size 1.5 1.5) (thickness 0.3)))
+  )
   (gr_text "Iwasz 2016" (at 117.475 84.455) (layer B.Cu)

Commit message: 2017 improvements
Parts:
- removed C18, C19: 15pF, w_smd_cap:c_0603
- removed C20, C22, C23: 100nF, w_smd_cap:c_0603
- removed C21: 33nF, w_smd_cap:c_0603
- removed C24, C25: 10pF, w_smd_cap:c_0603
- removed C26: 1nF, w_smd_cap:c_0603
- removed C27: 2.2nF, w_smd_cap:c_0603
- removed C28: 1.8pF, w_smd_cap:c_0603
- removed C29: 1.2pF, w_smd_cap:c_0603
- removed D2: LED, w_indicators:led_5mm_red
- removed L1: 8.2nH, w_smd_resistors:r_0603
- removed L2: 3.9nH, w_smd_resistors:r_0603
- removed L3: 5.6nH, w_smd_resistors:r_0603
- removed Q2, Q4: BC847, w_smd_trans:sot23
- removed Q5: NX7002AK, iwasz:sot23-pins123-ccw
- removed R10, R11, R12, R14, R15, R16, R17, R18, R19, R6, R7, R8: 33k, w_smd_resistors:r_0603
- removed R20, R33: 1k, w_smd_resistors:r_0603
- removed R21: 560R, w_smd_resistors:r_0603
- removed R29: 22k, w_smd_resistors:r_0603
- removed R30: AMCA31, w_smd_resistors:r_1206
- removed R34: 10k, w_smd_resistors:r_0603
- removed Y2: 32kHz, Crystals:Crystal_Round_Vertical_3mm
- removed Y3: 16MHz, w_crystal:crystal_hc-49s
- added J1: CONN_01X01, Mounting_Holes:MountingHole_3.2mm_M3_DIN965_Pad, B.Cu at (133.7, 124.6)
- added J10: CONN_01X01, Mounting_Holes:MountingHole_3.2mm_M3_DIN965_Pad, B.Cu at (133.8, 80.4)
- added J11: CONN_01X01, Mounting_Holes:MountingHole_3.2mm_M3_DIN965_Pad, B.Cu at (169.8, 80.4)
- added J12: CONN_01X01, Mounting_Holes:MountingHole_3.2mm_M3_DIN965_Pad, B.Cu at (169.8, 124.6)
- added J2: CONN_01X01, Pin_Headers:Pin_Header_Straight_1x01_Pitch2.00mm, B.Cu at (113.7, 79.4)
- added J3: CONN_01X01, Pin_Headers:Pin_Header_Straight_1x01_Pitch2.00mm, B.Cu at (164.5, 79.4)
- added J4: CONN_01X01, Pin_Headers:Pin_Header_Straight_1x01_Pitch2.00mm, B.Cu at (139.7, 79.4)
- added J5: CONN_01X01, Pin_Headers:Pin_Header_Straight_1x01_Pitch2.00mm, B.Cu at (190.5, 79.4)
- added J6: CONN_01X01, Pin_Headers:Pin_Header_Straight_1x01_Pitch2.00mm, B.Cu at (190.5, 125.7)
- added J7: CONN_01X01, Pin_Headers:Pin_Header_Straight_1x01_Pitch2.00mm, B.Cu at (164.5, 125.7)
- added J8: CONN_01X01, Pin_Headers:Pin_Header_Straight_1x01_Pitch2.00mm, B.Cu at (113.7, 125.7)
- added J9: CONN_01X01, Pin_Headers:Pin_Header_Straight_1x01_Pitch2.00mm, B.Cu at (139.7, 125.7)
- C16, C17: value 10µF -> 1µF, X5R, X7R, 25V; footprint w_smd_cap:c_tant_B -> w_smd_cap:c_0603
- P3: footprint w_pin_strip:pin_strip_4 -> w_pin_strip:pin_strip_2mm_4
- P6: value test-double -> CONN_01X04; footprint iwasz:testpad-2p -> w_pin_strip:pin_strip_2mm_4
- R1, R2: value 33k -> 10k
- R13: value 100R -> 1R
- R22: value R -> 220R
- R4, R5: value 33k -> 5k6
- U3: value STM32F0-LQFP48 -> STM32F072CB / STM32F042C6
- U6: value AP1117D33 -> MIC5504; footprint w_smd_trans:sot223 -> w_smd_trans:sot23-5
- U7: value nRF8001 -> PCF85176T; footprint w_smd_qfn:pvqfn-n32 -> micro-philips:TSSOP56-6
- Y1: value Crystal -> 8MHz
- moved R2 64.4 mm to (184.7, 97.3), turned to 0 degrees
- moved P3 44.8 mm to (154.7, 81.5)
- moved R4 44.6 mm to (167.1, 88.1), turned to 180 degrees
- moved R1 44.3 mm to (160.0, 106.9), turned to 90 degrees
- moved R5 42.4 mm to (167.1, 85.9), turned to 0 degrees
- moved C16 39.0 mm to (189.7, 111.0), turned to 90 degrees
- moved R31 38.1 mm to (153.7, 85.1), turned to 90 degrees
- moved R32 37.9 mm to (158.0, 85.1), turned to 90 degrees
- moved C17 36.5 mm to (182.4, 111.0), turned to 270 degrees
- moved SW2 31.1 mm to (184.9, 106.2), turned to 0 degrees
- moved U6 30.9 mm to (185.9, 110.7), turned to 0 degrees
- moved C2 30.4 mm to (164.6, 106.2)
- moved C5 30.0 mm to (164.6, 108.5)
- moved P6 26.8 mm to (180.6, 81.0)
- moved U3 22.2 mm to (159.5, 98.8), turned to 90 degrees
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Connections:
- net complete renamed /Sheet56372EC5/complete
- net progress renamed /Sheet56372EC5/progress
- P2 pad 1: Net-(P2-Pad1) -> /nrst
- P6 pad 1: Net-(P6-Pad1) -> /consoleTx
- R1 pad 1: +BATT -> Net-(R1-Pad1)
- R1 pad 2: /com1 -> GND
- R2 pad 1: +BATT -> GND
- R2 pad 2: /com2 -> Net-(P1-Pad2)
- R4 pad 1: +BATT -> /sense
- R4 pad 2: /com3 -> +BATT
- R5 pad 1: +BATT -> GND
- R5 pad 2: /com4 -> /sense
- R9 pad 2: +3V3 -> +BATT
- SP1 pad 1: +3V3 -> +BATT
- U2 pad 1: /com1 -> Net-(U2-Pad1)
- U2 pad 10: /seg6 -> Net-(U2-Pad10)
- U2 pad 11: /seg7 -> Net-(U2-Pad11)
- U2 pad 12: /seg8 -> Net-(U2-Pad12)
- U2 pad 13: /seg9 -> Net-(U2-Pad13)
- U2 pad 14: /seg10 -> Net-(U2-Pad14)
- U2 pad 15: /seg11 -> Net-(U2-Pad15)
- U2 pad 16: /seg12 -> Net-(U2-Pad16)
- U2 pad 2: /com2 -> Net-(U2-Pad2)
- U2 pad 3: /com3 -> Net-(U2-Pad3)
- U2 pad 4: /com4 -> Net-(U2-Pad4)
- U2 pad 5: /seg1 -> Net-(U2-Pad5)
- U2 pad 6: /seg2 -> Net-(U2-Pad6)
- U2 pad 7: /seg3 -> Net-(U2-Pad7)
- U2 pad 8: /seg4 -> Net-(U2-Pad8)
- U2 pad 9: /seg5 -> Net-(U2-Pad9)
- U3 pad 1: (no net) -> Net-(U3-Pad1)
- U3 pad 10: /indicator -> Net-(U3-Pad10)
- U3 pad 12: ble_active -> Net-(U3-Pad12)
- U3 pad 13: ble_reset -> /sense
- U3 pad 14: ble_reqn -> Net-(U3-Pad14)
- U3 pad 15: ble_sck -> Net-(U3-Pad15)
- U3 pad 16: ble_miso -> Net-(U3-Pad16)
- U3 pad 17: ble_mosi -> Net-(U3-Pad17)
- U3 pad 18: ble_rdyn -> Net-(U3-Pad18)
- U3 pad 20: /com1 -> Net-(U3-Pad20)
- U3 pad 21: /com2 -> Net-(U3-Pad21)
- U3 pad 22: /com3 -> Net-(U3-Pad22)
- U3 pad 25: /com4 -> Net-(U3-Pad25)
- U3 pad 26: /seg1 -> Net-(U3-Pad26)
- U3 pad 27: /seg2 -> Net-(U3-Pad27)
- U3 pad 28: /seg3 -> Net-(U3-Pad28)
- U3 pad 29: /seg4 -> Net-(U3-Pad29)
- U3 pad 30: /seg5 -> /consoleTx
- U3 pad 31: /seg6 -> /consoleRx
- U3 pad 38: /seg7 -> Net-(U3-Pad38)
- U3 pad 39: /seg8 -> Net-(U3-Pad39)
- U3 pad 40: /seg9 -> Net-(U3-Pad40)
- U3 pad 41: /seg10 -> Net-(U3-Pad41)
- U3 pad 42: /seg11 -> /screen/scl
- U3 pad 43: /seg12 -> /screen/sda
- U3 pad 44: (no net) -> Net-(R1-Pad1)
- U3 pad 7: Net-(P2-Pad1) -> /nrst
- U4 pad 4: (no net) -> Net-(U4-Pad4)
- U5 pad 7: Net-(P6-Pad1) -> Net-(U5-Pad7)
- U6 pad 1: GND -> +BATT
- U6 pad 2: +3V3 -> GND
- U7 pad 1: +3V3 -> Net-(U2-Pad3)
- U7 pad 10: (no net) -> Net-(U2-Pad11)
- U7 pad 11: ble_sck -> Net-(U2-Pad12)
- U7 pad 12: ble_reqn -> Net-(U2-Pad13)
- U7 pad 13: ble_mosi -> Net-(U2-Pad14)
- U7 pad 14: ble_miso -> Net-(U2-Pad15)
- U7 pad 15: (no net) -> Net-(U2-Pad16)
- U7 pad 16: ble_rdyn -> Net-(U7-Pad16)
- U7 pad 17: GND -> Net-(U7-Pad17)
- U7 pad 18: GND -> Net-(U7-Pad18)
- U7 pad 19: ble_reset -> Net-(U7-Pad19)
- U7 pad 2: Net-(C20-Pad1) -> Net-(U2-Pad2)
- U7 pad 23: GND -> Net-(U7-Pad23)
- U7 pad 24: +3V3 -> Net-(U7-Pad24)
- U7 pad 26: +3V3 -> Net-(U7-Pad26)
- U7 pad 29: +3V3 -> Net-(U7-Pad29)
- U7 pad 3: Net-(C21-Pad1) -> Net-(U2-Pad4)
- U7 pad 30: GND -> Net-(U7-Pad30)
- U7 pad 31: GND -> Net-(U7-Pad31)
- U7 pad 32: (no net) -> Net-(U7-Pad32)
- U7 pad 33: GND -> Net-(U7-Pad33)
- U7 pad 4: Net-(C18-Pad1) -> Net-(U2-Pad5)
- U7 pad 5: Net-(C19-Pad1) -> Net-(U2-Pad6)
- U7 pad 6: ble_active -> Net-(U2-Pad7)
- U7 pad 7: (no net) -> Net-(U2-Pad8)
- U7 pad 8: GND -> Net-(U2-Pad9)
- U7 pad 9: +3V3 -> Net-(U2-Pad10)
Routing:
- net GND: track 1143.3 -> 412.8 mm, vias 233 -> 77
- net /nrst: track 0.00 -> 46.1 mm, vias 0 -> 2
- net /indicator: track 44.5 -> 0.00 mm, vias 2 -> 0
- net /screen/scl: track 0.00 -> 37.3 mm, vias 0 -> 2
- net /screen/sda: track 0.00 -> 35.8 mm, vias 0 -> 2
- net Net-(P6-Pad1): track 29.5 -> 0.00 mm
- net +3V3: track 183.7 -> 154.6 mm, vias 14 -> 3
- net /ir: track 31.5 -> 60.4 mm, vias 2 -> 0
- net Net-(R23-Pad2): track 58.0 -> 29.3 mm
- net Net-(P1-Pad1): track 40.1 -> 13.0 mm
- net Net-(R24-Pad2): track 56.1 -> 29.2 mm
- net Net-(U2-Pad16): track 0.00 -> 26.6 mm
- net /seg12: track 26.5 -> 0.00 mm, vias 2 -> 0
- net /seg11: track 25.7 -> 0.00 mm, vias 4 -> 0
- net /consoleRx: track 0.00 -> 25.5 mm
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Other:
- outline, holes or cut-outs redrawn
- board text added: "1"
- board text added: "Iwasz 2017"
- board text added: "T"
- board text added: "moto-gymkhana stopwatch by iwasz. rev3. 2017"
- board text added: "nrst"
- board text added: "rx"
- board text added: "tx"
- board text removed: "Iwasz 2016"
- board text removed: "moto-gymkhana stopwatch by iwasz. rev2. 2016"
