File: hw-design/receiver/screen.sch (KiCad schematic (older format))
At the start: 2 parts, among them U2 weight-scale-lcd, U7 PCF85176T

Commit message: Many changes
Parts:
- U2: symbol weight-scale-lcd -> iwasz-kicad:weight-scale-lcd
- U7: symbol PCF85176T -> iwasz-kicad:PCF85176T
Changed lines of the file:
@@
-EESchema Schematic File Version 2
-LIBS:iwasz-kicad
-LIBS:power
-LIBS:device
-LIBS:transistors
-LIBS:conn
-LIBS:linear
-LIBS:regul
-LIBS:74xx
-LIBS:cmos4000
-LIBS:adc-dac
-LIBS:memory
-LIBS:xilinx
-LIBS:microcontrollers
-LIBS:dsp
-LIBS:microchip
-LIBS:analog_switches
-LIBS:motorola
-LIBS:texas
-LIBS:intel
-LIBS:audio
-LIBS:interface
-LIBS:digital-audio
-LIBS:philips
-LIBS:display
-LIBS:cypress
-LIBS:siliconi
-LIBS:opto
-LIBS:atmel
-LIBS:contrib
-LIBS:valves
+EESchema Schematic File Version 4
 LIBS:gp8-clock-cache
 EELAYER 26 0
@@
 $Descr A4 11693 8268
 encoding utf-8
-Sheet 3 3
+Sheet 2 2
 Title ""
 Date ""
@@
 $EndDescr
 $Comp
-L weight-scale-lcd U2
+L iwasz-kicad:weight-scale-lcd U2
 U 1 1 58BEC91B
 P 4400 1950
@@
 LCD screen
 $Comp
-L PCF85176T U7
+L iwasz-kicad:PCF85176T U7
 U 1 1 58BEC923
 P 6200 4175
@@
 NoConn ~ 6900 4225
 $Comp
-L GND #PWR036
+L power:GND #PWR036
 U 1 1 58BEC967
 P 7075 3125
@@
 $EndComp
 Wire Wire Line
-	6900 3125 7075 3125
+	6900 3125 7000 3125
 Wire Wire Line
 	6900 3225 7000 3225
 Wire Wire Line
-	7000 3125 7000 3625
+	7000 3125 7000 3225
 Connection ~ 7000 3125
 Wire Wire Line
@@
 NoConn ~ 6900 3825
 $Comp
-L +3.3V #PWR037
+L power:+3.3V #PWR037
 U 1 1 58BEC980
 P 6975 3025
@@
 	6900 3025 6975 3025
 $Comp
-L +3.3V #PWR038
+L power:+3.3V #PWR038
 U 1 1 58BEC987
 P 6975 3725
@@
 Text HLabel 6900 4125 2    60   BiDi ~ 0
 sda
+Wire Wire Line
+	7000 3125 7075 3125
+Wire Wire Line
+	7000 3225 7000 3325
+Wire Wire Line
+	7000 3325 7000 3425
+Wire Wire Line
+	7000 3425 7000 3525
+Wire Wire Line
+	7000 3525 7000 3625
 $EndSCHEMATC
